File: pcbservo-dc/untitled.kicad_sch1.kicad_sch (KiCad schematic)
At the start: 21 parts, among them J1 Conn_01x02, J14 R-78B5.0-2.0, J2 Conn_01x02, J3 BU33SD5WG-TR

Commit message: changement de quelques empreinte
Parts:
- J1, J2: footprint Connector_JST:JST_XH_B2B-XH-A_1x02_P2.50mm_Vertical -> Connector_JST:JST_EH_B2B-EH-A_1x02_P2.50mm_Vertical
Changed lines of the file:
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@@
 			)
 		)
-		(property "Footprint" "Connector_JST:JST_XH_B2B-XH-A_1x02_P2.50mm_Vertical"
+		(property "Footprint" "Connector_JST:JST_EH_B2B-EH-A_1x02_P2.50mm_Vertical"
 			(at 123.19 54.61 0)
 			(effects
@@
 			)
 		)
-		(property "Footprint" "Connector_JST:JST_XH_B2B-XH-A_1x02_P2.50mm_Vertical"
+		(property "Footprint" "Connector_JST:JST_EH_B2B-EH-A_1x02_P2.50mm_Vertical"
 			(at 119.38 26.67 0)
 			(effects
